Commit message: test

File: arm_ws/src/d2_moveit/config/gazebo_robot_arm.urdf (robot description, URDF)
Before this commit: robot robot_arm, 8 links, 7 joints
Links:
- link gripper_2: geometry collision sphere radius=0.00; visual sphere radius=0.00

File: arm_ws/src/robot_arm_description/urdf/robot_arm.xacro (robot description, xacro)
@@ -4,5 +4,5 @@
 <xacro:include filename="$(find robot_arm_description)/urdf/robot_arm.trans" />
 <xacro:include filename="$(find robot_arm_description)/urdf/robot_arm.gazebo" />
-<!--<link name="world"/>-->
+<link name="world"/>
 <link name="base_link">
   <inertial>
@@ -122,10 +122,10 @@
 <link name="gripper_2">
   <inertial>
-    <origin xyz="0.04 0.0 0.05" rpy="0 0 0"/>
+    <origin xyz="0.0 0.0 0.0" rpy="0 0 0"/>
     <mass value="0.0"/>
     <inertia ixx="0" iyy="0" izz="0" ixy="0" iyz="0" ixz="0"/>
   </inertial>
   <visual>
-    <origin xyz="0.04 0.0 0.05" rpy="0 0 0"/>
+    <origin xyz="0.0 0.0 0.0" rpy="0 0 0"/>
     <geometry>
       <sphere radius="0.01"/>
@@ -133,5 +133,5 @@
   </visual>
   <collision>
-    <origin xyz="0.04 0.0 0.05" rpy="0 0 0"/>
+    <origin xyz="0.0 0.0 0.0" rpy="0 0 0"/>
     <geometry>
       <sphere radius="0.00"/>
@@ -174,15 +174,16 @@
   <limit upper="1.570796" lower="-1.570796" effort="1.075" velocity="6"/>
 </joint>
-<!--<joint name="fixed" type="fixed">
+<joint name="fixed" type="fixed">
     <parent link="world"/>
     <child link="base_link"/>
     <origin xyz="0.0 0.0 0.0" rpy="0 0 0"/>
-  </joint>-->
-<joint name="end_eff" type="revolute">
+  </joint>
+<joint name="end_eff" type="fixed">
+    <!--<origin xyz="0.076264 -0.005 0.093335" rpy="0 0 0"/>-->
     <origin xyz="0.076264 0.005 0.093335" rpy="0 0 0"/>
     <parent link="gripper_1"/>
     <child link="gripper_2"/>
     <axis xyz="-0.0 -1.0 0.0"/>
-    <limit upper="1.570796" lower="-1.570796" effort="1.075" velocity="6"/>
+    <!--<limit upper="1.570796" lower="-1.570796" effort="1.075" velocity="6"/>-->
 </joint>
 </robot>

File: arm_ws/src/robot_arm_moveit/config/gazebo_robot_arm.urdf (robot description, URDF)
Before this commit: robot robot_arm, 7 links, 6 joints
Links:
- added link gripper_2, mass 0.0; collision sphere radius=0.00; visual sphere radius=0.00
Joints:
- added joint end_eff: type revolute, parent gripper_1, child gripper_2, origin xyz=0.076264 0.005 0.093335 rpy=0 0 0, axis -0.0 -1.0 0.0, limit lower=-1.570796 upper=1.570796 effort=1.075 velocity=6

Commit message: test

File: arm_ws/src/d2_moveit/config/gazebo_robot_arm.urdf (robot description, URDF)
Before this commit: robot robot_arm, 8 links, 7 joints
Links:
- link gripper_2: geometry collision sphere radius=0.00; visual sphere radius=0.01
Joints:
- joint end_eff: limit lower=-1.570796 upper=1.570796 effort=1.075 velocity=6 -> (none); type revolute -> fixed

File: arm_ws/src/robot_arm_description/urdf/robot_arm.xacro (robot description, xacro)
@@ -123,6 +123,6 @@
   <inertial>
     <origin xyz="0.0 0.0 0.0" rpy="0 0 0"/>
-    <mass value="0.0"/>
-    <inertia ixx="0" iyy="0" izz="0" ixy="0" iyz="0" ixz="0"/>
+    <mass value="0.00001"/>
+    <inertia ixx="0.0" iyy="0.0" izz="0.0" ixy="0.0" iyz="0.0" ixz="0.0"/>
   </inertial>
   <visual>
@@ -144,5 +144,5 @@
   <child link="waist_1"/>
   <axis xyz="-0.0 0.0 1.0"/>
-  <limit upper="1.570796" lower="-1.570796" effort="1.075" velocity="6"/>
+  <limit upper="1.570796" lower="-1.570796" effort="1.075" velocity="1000"/>
 </joint>
 <joint name="waist_joint" type="revolute">
@@ -151,5 +151,5 @@
   <child link="arm1_1"/>
   <axis xyz="0.0 -1.0 0.0"/>
-  <limit upper="1.570796" lower="-1.27409" effort="1.075" velocity="6"/>
+  <limit upper="1.570796" lower="-1.27409" effort="1.075" velocity="1000"/>
 </joint>
 <joint name="arm1_joint" type="revolute">
@@ -158,5 +158,5 @@
   <child link="arm2_1"/>
   <axis xyz="-0.0 1.0 -0.0"/>
-  <limit upper="1.570796" lower="-1.570796" effort="1.075" velocity="6"/>
+  <limit upper="1.570796" lower="-1.570796" effort="1.075" velocity="1000"/>
 </joint>
 <joint name="arm2_joint" type="revolute">
@@ -165,5 +165,5 @@
   <child link="arm3_1"/>
   <axis xyz="0.707107 0.0 0.707107"/>
-  <limit upper="1.570796" lower="-1.570796" effort="1.075" velocity="6"/>
+  <limit upper="1.570796" lower="-1.570796" effort="1.075" velocity="1000"/>
 </joint>
 <joint name="arm3_joint" type="revolute">
@@ -172,5 +172,5 @@
   <child link="gripper_1"/>
   <axis xyz="-0.0 -1.0 0.0"/>
-  <limit upper="1.570796" lower="-1.570796" effort="1.075" velocity="6"/>
+  <limit upper="1.570796" lower="-1.570796" effort="1.075" velocity="1000"/>
 </joint>
 <joint name="fixed" type="fixed">
@@ -179,5 +179,5 @@
     <origin xyz="0.0 0.0 0.0" rpy="0 0 0"/>
   </joint>
-<joint name="end_eff" type="fixed">
+<joint name="end_eff" type="revolute">
     <!--<origin xyz="0.076264 -0.005 0.093335" rpy="0 0 0"/>-->
     <origin xyz="0.076264 0.005 0.093335" rpy="0 0 0"/>
@@ -185,5 +185,5 @@
     <child link="gripper_2"/>
     <axis xyz="-0.0 -1.0 0.0"/>
-    <!--<limit upper="1.570796" lower="-1.570796" effort="1.075" velocity="6"/>-->
+    <limit upper="1.570796" lower="-1.570796" effort="1.075" velocity="1000"/>
 </joint>
 </robot>
