Commit message: Update urdf

File: arm_ws/src/robot_arm_description/urdf/robot_arm.xacro (robot description, xacro)
@@ -120,5 +120,5 @@
   </collision>
 </link>
-<link name="gripper_2">
+<!--<link name="gripper_2">
   <inertial>
     <origin xyz="0.04 0.0 0.05" rpy="0 0 0"/>
@@ -138,5 +138,5 @@
     </geometry>
   </collision>
-</link>
+</link>-->
 <joint name="base_joint" type="revolute">
   <origin xyz="0.0 0.0 0.0566" rpy="0 0 0"/>
@@ -179,9 +179,9 @@
     <origin xyz="0.0 0.0 0.0" rpy="0 0 0"/>
   </joint>
-  <joint name="fixed2" type="fixed">
+  <!--<joint name="fixed2" type="fixed">
     <origin xyz="0.036264 0.005 0.043335" rpy="0 0 0"/>
     <parent link="gripper_1"/>
     <child link="gripper_2"/>
     <axis xyz="-0.0 -1.0 0.0"/>
-  </joint>
+  </joint>-->
 </robot>

Commit message: MoveIt

File: arm_ws/src/robot_arm_description/urdf/robot_arm.xacro (robot description, xacro)
@@ -120,5 +120,5 @@
   </collision>
 </link>
-<!--<link name="gripper_2">
+<link name="gripper_2">
   <inertial>
     <origin xyz="0.04 0.0 0.05" rpy="0 0 0"/>
@@ -129,5 +129,5 @@
     <origin xyz="0.04 0.0 0.05" rpy="0 0 0"/>
     <geometry>
-      <sphere radius="0.01"/>
+      <sphere radius="0.00"/>
     </geometry>
   </visual>
@@ -135,8 +135,8 @@
     <origin xyz="0.04 0.0 0.05" rpy="0 0 0"/>
     <geometry>
-      <sphere radius="0.01"/>
+      <sphere radius="0.00"/>
     </geometry>
   </collision>
-</link>-->
+</link>
 <joint name="base_joint" type="revolute">
   <origin xyz="0.0 0.0 0.0566" rpy="0 0 0"/>
@@ -179,9 +179,9 @@
     <origin xyz="0.0 0.0 0.0" rpy="0 0 0"/>
   </joint>
-  <!--<joint name="fixed2" type="fixed">
-    <origin xyz="0.036264 0.005 0.043335" rpy="0 0 0"/>
+  <joint name="fixed2" type="fixed">
+    <origin xyz="0.076264 0.005 0.093335" rpy="0 0 0"/>
     <parent link="gripper_1"/>
     <child link="gripper_2"/>
     <axis xyz="-0.0 -1.0 0.0"/>
-  </joint>-->
+  </joint>
 </robot>

Commit message: Moveit

File: arm_ws/src/robot_arm_description/urdf/robot_arm.xacro (robot description, xacro)
@@ -120,5 +120,5 @@
   </collision>
 </link>
-<link name="gripper_2">
+<!--<link name="gripper_2">
   <inertial>
     <origin xyz="0.04 0.0 0.05" rpy="0 0 0"/>
@@ -138,5 +138,5 @@
     </geometry>
   </collision>
-</link>
+</link>-->
 <joint name="base_joint" type="revolute">
   <origin xyz="0.0 0.0 0.0566" rpy="0 0 0"/>
@@ -179,9 +179,9 @@
     <origin xyz="0.0 0.0 0.0" rpy="0 0 0"/>
   </joint>
-  <joint name="fixed2" type="fixed">
+<!--<joint name="fixed2" type="fixed">
     <origin xyz="0.076264 0.005 0.093335" rpy="0 0 0"/>
     <parent link="gripper_1"/>
     <child link="gripper_2"/>
     <axis xyz="-0.0 -1.0 0.0"/>
-  </joint>
+</joint>-->
 </robot>

File: arm_ws/src/robot_arm_moveit/config/gazebo_robot_arm.urdf (robot description, URDF)
Before this commit: robot robot_arm, 8 links, 7 joints
Links:
- removed link gripper_2
Joints:
- removed joint fixed2

Commit message: test

File: arm_ws/src/robot_arm_description/urdf/robot_arm.xacro (robot description, xacro)
@@ -4,5 +4,5 @@
 <xacro:include filename="$(find robot_arm_description)/urdf/robot_arm.trans" />
 <xacro:include filename="$(find robot_arm_description)/urdf/robot_arm.gazebo" />
-<link name="world"/>
+<!--<link name="world"/>-->
 <link name="base_link">
   <inertial>
@@ -120,5 +120,5 @@
   </collision>
 </link>
-<!--<link name="gripper_2">
+<link name="gripper_2">
   <inertial>
     <origin xyz="0.04 0.0 0.05" rpy="0 0 0"/>
@@ -129,5 +129,5 @@
     <origin xyz="0.04 0.0 0.05" rpy="0 0 0"/>
     <geometry>
-      <sphere radius="0.00"/>
+      <sphere radius="0.01"/>
     </geometry>
   </visual>
@@ -138,5 +138,5 @@
     </geometry>
   </collision>
-</link>-->
+</link>
 <joint name="base_joint" type="revolute">
   <origin xyz="0.0 0.0 0.0566" rpy="0 0 0"/>
@@ -174,14 +174,15 @@
   <limit upper="1.570796" lower="-1.570796" effort="1.075" velocity="6"/>
 </joint>
-<joint name="fixed" type="fixed">
+<!--<joint name="fixed" type="fixed">
     <parent link="world"/>
     <child link="base_link"/>
     <origin xyz="0.0 0.0 0.0" rpy="0 0 0"/>
-  </joint>
-<!--<joint name="fixed2" type="fixed">
+  </joint>-->
+<joint name="end_eff" type="revolute">
     <origin xyz="0.076264 0.005 0.093335" rpy="0 0 0"/>
     <parent link="gripper_1"/>
     <child link="gripper_2"/>
     <axis xyz="-0.0 -1.0 0.0"/>
-</joint>-->
+    <limit upper="1.570796" lower="-1.570796" effort="1.075" velocity="6"/>
+</joint>
 </robot>

Commit message: test2

File: arm_ws/src/robot_arm_description/urdf/robot_arm.xacro (robot description, xacro)
@@ -123,5 +123,5 @@
   <inertial>
     <origin xyz="0.0 0.0 0.0" rpy="0 0 0"/>
-    <mass value="0.00001"/>
+    <mass value="0.0"/>
     <inertia ixx="0.0" iyy="0.0" izz="0.0" ixy="0.0" iyz="0.0" ixz="0.0"/>
   </inertial>

Commit message: web app

File: arm_ws/src/robot_arm_description/urdf/robot_arm.xacro (robot description, xacro)
@@ -144,5 +144,5 @@
   <child link="waist_1"/>
   <axis xyz="-0.0 0.0 1.0"/>
-  <limit upper="1.570796" lower="-1.570796" effort="1.075" velocity="1000"/>
+  <limit upper="1.570796" lower="-1.570796" effort="15.075" velocity="2"/>
 </joint>
 <joint name="waist_joint" type="revolute">
@@ -151,5 +151,5 @@
   <child link="arm1_1"/>
   <axis xyz="0.0 -1.0 0.0"/>
-  <limit upper="1.570796" lower="-1.27409" effort="1.075" velocity="1000"/>
+  <limit upper="1.570796" lower="-1.27409" effort="15.075" velocity="2"/>
 </joint>
 <joint name="arm1_joint" type="revolute">
@@ -158,5 +158,5 @@
   <child link="arm2_1"/>
   <axis xyz="-0.0 1.0 -0.0"/>
-  <limit upper="1.570796" lower="-1.570796" effort="1.075" velocity="1000"/>
+  <limit upper="1.570796" lower="-1.570796" effort="15.075" velocity="2"/>
 </joint>
 <joint name="arm2_joint" type="revolute">
@@ -165,5 +165,5 @@
   <child link="arm3_1"/>
   <axis xyz="0.707107 0.0 0.707107"/>
-  <limit upper="1.570796" lower="-1.570796" effort="1.075" velocity="1000"/>
+  <limit upper="1.570796" lower="-1.570796" effort="15.075" velocity="2"/>
 </joint>
 <joint name="arm3_joint" type="revolute">
@@ -172,5 +172,5 @@
   <child link="gripper_1"/>
   <axis xyz="-0.0 -1.0 0.0"/>
-  <limit upper="1.570796" lower="-1.570796" effort="1.075" velocity="1000"/>
+  <limit upper="1.570796" lower="-1.570796" effort="15.075" velocity="2"/>
 </joint>
 <joint name="fixed" type="fixed">
@@ -185,5 +185,5 @@
     <child link="gripper_2"/>
     <axis xyz="-0.0 -1.0 0.0"/>
-    <limit upper="1.570796" lower="-1.570796" effort="1.075" velocity="1000"/>
+    <limit upper="1.570796" lower="-1.570796" effort="15.075" velocity="2"/>
 </joint>
 </robot>

Commit message: test

File: arm_ws/src/robot_arm_description/urdf/robot_arm.xacro (robot description, xacro)
@@ -144,5 +144,5 @@
   <child link="waist_1"/>
   <axis xyz="-0.0 0.0 1.0"/>
-  <limit upper="1.570796" lower="-1.570796" effort="15.075" velocity="2"/>
+  <limit upper="1.570796" lower="-1.570796" effort="1.075" velocity="2"/>
 </joint>
 <joint name="waist_joint" type="revolute">
@@ -151,5 +151,5 @@
   <child link="arm1_1"/>
   <axis xyz="0.0 -1.0 0.0"/>
-  <limit upper="1.570796" lower="-1.27409" effort="15.075" velocity="2"/>
+  <limit upper="1.570796" lower="-1.27409" effort="1.075" velocity="2"/>
 </joint>
 <joint name="arm1_joint" type="revolute">
@@ -158,5 +158,5 @@
   <child link="arm2_1"/>
   <axis xyz="-0.0 1.0 -0.0"/>
-  <limit upper="1.570796" lower="-1.570796" effort="15.075" velocity="2"/>
+  <limit upper="1.570796" lower="-1.570796" effort="1.075" velocity="2"/>
 </joint>
 <joint name="arm2_joint" type="revolute">
@@ -165,5 +165,5 @@
   <child link="arm3_1"/>
   <axis xyz="0.707107 0.0 0.707107"/>
-  <limit upper="1.570796" lower="-1.570796" effort="15.075" velocity="2"/>
+  <limit upper="1.570796" lower="-1.570796" effort="1.075" velocity="2"/>
 </joint>
 <joint name="arm3_joint" type="revolute">
@@ -172,5 +172,5 @@
   <child link="gripper_1"/>
   <axis xyz="-0.0 -1.0 0.0"/>
-  <limit upper="1.570796" lower="-1.570796" effort="15.075" velocity="2"/>
+  <limit upper="1.570796" lower="-1.570796" effort="1.075" velocity="2"/>
 </joint>
 <joint name="fixed" type="fixed">
@@ -185,5 +185,5 @@
     <child link="gripper_2"/>
     <axis xyz="-0.0 -1.0 0.0"/>
-    <limit upper="1.570796" lower="-1.570796" effort="15.075" velocity="2"/>
+    <limit upper="1.570796" lower="-1.570796" effort="1.075" velocity="2"/>
 </joint>
 </robot>
